Commit message: fix gripper

File: simulation/gazebo/arm_sim_scenario/urdf/wx200.urdf.xacro (robot description, xacro)
@@ -42,5 +42,5 @@
   <xacro:property name="gripper_limit_vel"          value="${pi}"/>
   <xacro:property name="finger_limit_effort"        value="5"/>
-  <xacro:property name="finger_limit_lower"         value="0.015"/>
+  <xacro:property name="finger_limit_lower"         value="-0.037"/>
   <xacro:property name="finger_limit_upper"         value="0.037"/>
   <xacro:property name="finger_limit_vel"           value="1"/>
