Commit message: description cleanup

File: simulation/gazebo/arm_sim_scenario/urdf/control.urdf.xacro (robot description, xacro)
@@ -16,8 +16,11 @@
       </xacro:if>
       <!-- If simulating the robot in Gazebo Classic -->
-      <!-- <xacro:if value="${hardware_type == 'gz_classic'}"> -->
-        <!-- <plugin>gazebo_ros2_control/GazeboSystem</plugin> -->
-      <plugin>ign_ros2_control/IgnitionSystem</plugin>
-      <!-- </xacro:if> -->
+      <xacro:if value="${hardware_type == 'gz_classic'}">
+        <plugin>gazebo_ros2_control/GazeboSystem</plugin>
+      </xacro:if>
+    <!-- If simulating the robot in Gazebo Modern -->
+      <xacro:if value="${hardware_type == 'ignition'}">
+        <plugin>ign_ros2_control/IgnitionSystem</plugin>
+      </xacro:if>
     </hardware>
     <joint name="waist">
@@ -68,10 +71,10 @@
     </xacro:if>
     <xacro:if value="$(arg use_gripper)">
-      <!-- <xacro:if value="${hardware_type in ('fake', 'gz_classic')}"> -->
-      <joint name="gripper">
-        <command_interface name="position"/>
-        <state_interface name="position"/>
-      </joint>
-      <!-- </xacro:if> -->
+      <xacro:if value="${hardware_type in ('fake', 'gz_classic', 'ignition')}">
+        <joint name="gripper">
+          <command_interface name="position"/>
+          <state_interface name="position"/>
+        </joint>
+      </xacro:if>
       <xacro:if value="$(arg show_gripper_fingers)">
         <joint name="left_finger">
@@ -82,5 +85,5 @@
           <state_interface name="position"/>
         </joint>
-        <!-- <xacro:if value="${hardware_type == 'gz_classic'}"> -->
+        <xacro:if value="${hardware_type in ('gz_classic', 'ignition')}">
           <joint name="right_finger">
             <!-- <param name="mimic">left_finger</param>
@@ -92,21 +95,34 @@
             <state_interface name="position"/>
           </joint>
-        <!-- </xacro:if> -->
+        </xacro:if>
       </xacro:if>
     </xacro:if>
   </ros2_control>
   <!-- Load the gazebo_ros2_control plugin if using Gazebo hardware -->
-  <!-- <xacro:if value="${hardware_type == 'gz_classic'}"> -->
-  <gazebo>
-    <plugin filename="libign_ros2_control-system.so" name="ign_ros2_control::IgnitionROS2ControlPlugin">
-      <ros>
-        <namespace>/$(arg robot_name)</namespace>
-      </ros>
-      <robot_param>robot_description</robot_param>
-      <robot_param_node>robot_state_publisher</robot_param_node>
-      <parameters>$(find arm_sim_scenario)/config/trajectory_controllers/${robot_model}_trajectory_controllers.yaml</parameters>
-    </plugin>
-  </gazebo>
-  <xacro:include filename="$(find arm_sim_scenario)/meshes/interbotix_texture.gazebo"/>
-  <!-- </xacro:if> -->
+  <xacro:if value="${hardware_type == 'gz_classic'}">
+    <gazebo>
+      <plugin filename="libgazebo_ros2_control.so" name="gazebo_ros2_control">
+        <ros>
+          <namespace>/$(arg robot_name)</namespace>
+        </ros>
+        <robot_param>robot_description</robot_param>
+        <robot_param_node>robot_state_publisher</robot_param_node>
+        <parameters>$(find arm_sim_scenario)/config/trajectory_controllers/${robot_model}_trajectory_controllers.yaml</parameters>
+      </plugin>
+    </gazebo>
+    <xacro:include filename="$(find arm_sim_scenario)/meshes/interbotix_texture.gazebo"/>
+  </xacro:if>
+  <xacro:if value="${hardware_type == 'ignition'}">
+    <gazebo>
+      <plugin filename="libign_ros2_control-system.so" name="ign_ros2_control::IgnitionROS2ControlPlugin">
+        <ros>
+          <namespace>/$(arg robot_name)</namespace>
+        </ros>
+        <robot_param>robot_description</robot_param>
+        <robot_param_node>robot_state_publisher</robot_param_node>
+        <parameters>$(find arm_sim_scenario)/config/trajectory_controllers/${robot_model}_trajectory_controllers.yaml</parameters>
+      </plugin>
+    </gazebo>
+    <xacro:include filename="$(find arm_sim_scenario)/meshes/interbotix_texture.gazebo"/>
+  </xacro:if>
 </robot>

File: simulation/gazebo/arm_sim_scenario/urdf/wx200.urdf.xacro (robot description, xacro)
@@ -15,5 +15,5 @@
   <xacro:arg name="use_world_frame"                 default="false"/>
   <xacro:arg name="external_urdf_loc"               default=""/>
-  <xacro:arg name="hardware_type"                   default="actual"/>
+  <xacro:arg name="hardware_type"                   default="ignition"/>
   <xacro:property name="mesh_directory"             value="package://arm_sim_scenario/meshes/${robot_model}_meshes"/>
   <xacro:property name="urdf_loc"                   value="$(arg external_urdf_loc)"/>
@@ -42,5 +42,5 @@
   <xacro:property name="gripper_limit_vel"          value="${pi}"/>
   <xacro:property name="finger_limit_effort"        value="5"/>
-  <xacro:property name="finger_limit_lower"         value="-0.037"/>
+  <xacro:property name="finger_limit_lower"         value="0.015"/>
   <xacro:property name="finger_limit_upper"         value="0.037"/>
   <xacro:property name="finger_limit_vel"           value="1"/>
@@ -586,5 +586,5 @@
             friction="0.1"
             damping="0.1"/>
-          <xacro:if value="${hardware_type != 'gz_classic'}">
+          <xacro:if value="${hardware_type not in ('ignition','gz_classic')}">
             <mimic
               joint="left_finger"
@@ -656,7 +656,7 @@
   <xacro:include filename="$(find arm_sim_scenario)/urdf/control.urdf.xacro"/>
   <xacro:include filename="$(find arm_sim_scenario)/urdf/gazebo_configs.urdf.xacro"/>
-  <!-- <xacro:if value="${hardware_type == 'gz_classic'}"> -->
+  <xacro:if value="${hardware_type == 'gz_classic'}">
     <xacro:gazebo_configs/>
-  <!-- </xacro:if> -->
+  </xacro:if>
   <xacro:if value="${urdf_loc != ''}">
     <xacro:include filename="${urdf_loc}"/>

Commit message: fix urdf

File: simulation/gazebo/arm_sim_scenario/urdf/control.urdf.xacro (robot description, xacro)
@@ -19,5 +19,5 @@
         <plugin>gazebo_ros2_control/GazeboSystem</plugin>
       </xacro:if>
-    <!-- If simulating the robot in Gazebo Modern -->
+      <!-- If simulating the robot in Gazebo Modern -->
       <xacro:if value="${hardware_type == 'ignition'}">
         <plugin>ign_ros2_control/IgnitionSystem</plugin>
@@ -29,5 +29,7 @@
         <param name="max">"${waist_limit_upper}"</param>
       </command_interface>
-      <state_interface name="position"/>
+      <state_interface name="position">
+        <param name="initial_value">${waist_initial_value}</param>
+      </state_interface>
     </joint>
     <joint name="shoulder">
@@ -36,5 +38,7 @@
         <param name="max">"${shoulder_limit_upper}"</param>
       </command_interface>
-      <state_interface name="position"/>
+      <state_interface name="position">
+        <param name="initial_value">${shoulder_initial_value}</param>
+      </state_interface>
     </joint>
     <joint name="elbow">
@@ -43,5 +47,7 @@
         <param name="max">"${elbow_limit_upper}"</param>
       </command_interface>
-      <state_interface name="position"/>
+      <state_interface name="position">
+        <param name="initial_value">${elbow_initial_value}</param>
+      </state_interface>
     </joint>
     <xacro:if value="${dof >= 6}">
@@ -51,5 +57,7 @@
           <param name="max">"${forearm_roll_limit_upper}"</param>
         </command_interface>
-        <state_interface name="position"/>
+        <state_interface name="position">
+          <param name="initial_value">${forearm_roll_initial_value}</param>
+        </state_interface>
       </joint>
     </xacro:if>
@@ -59,5 +67,7 @@
         <param name="max">"${wrist_angle_limit_upper}"</param>
       </command_interface>
-      <state_interface name="position"/>
+      <state_interface name="position">
+        <param name="initial_value">${wrist_angle_initial_value}</param>
+      </state_interface>
     </joint>
     <xacro:if value="${dof >= 5}">
@@ -65,5 +75,5 @@
         <command_interface name="position">
           <param name="min">"${wrist_rotate_limit_lower}"</param>
-          <param name="max">"${wrist_rotate_limit_upper}"</param>
+          <param name="max">${wrist_rotate_limit_upper}</param>
         </command_interface>
         <state_interface name="position"/>
@@ -84,5 +94,5 @@
           </command_interface>
           <state_interface name="position">
-            <param name="initial_value">0.0195</param>
+            <param name="initial_value">${finger_initial_value}</param>
           </state_interface>
         </joint>
@@ -95,7 +105,7 @@
               <param name="max">"${finger_limit_lower}"</param>
             </command_interface>
-          <state_interface name="position">
-            <param name="initial_value">-0.0195</param>
-          </state_interface>
+            <state_interface name="position">
+              <param name="initial_value">-${finger_initial_value}</param>
+            </state_interface>
           </joint>
         </xacro:if>
@@ -112,8 +122,8 @@
         <robot_param>robot_description</robot_param>
         <robot_param_node>robot_state_publisher</robot_param_node>
-        <parameters>$(find arm_sim_scenario)/config/trajectory_controllers/${robot_model}_trajectory_controllers.yaml</parameters>
+        <parameters>$(find interbotix_xsarm_sim)/config/trajectory_controllers/${robot_model}_trajectory_controllers.yaml</parameters>
       </plugin>
     </gazebo>
-    <xacro:include filename="$(find arm_sim_scenario)/meshes/interbotix_texture.gazebo"/>
+    <xacro:include filename="$(find interbotix_common_sim)/media/materials/scripts/interbotix_texture.gazebo"/>
   </xacro:if>
   <xacro:if value="${hardware_type == 'ignition'}">

File: simulation/gazebo/arm_sim_scenario/urdf/wx200.urdf.xacro (robot description, xacro)
@@ -15,5 +15,12 @@
   <xacro:arg name="use_world_frame"                 default="false"/>
   <xacro:arg name="external_urdf_loc"               default=""/>
-  <xacro:arg name="hardware_type"                   default="ignition"/>
+  <xacro:arg name="hardware_type"                   default="actual"/>
+  <!-- Initial values -->
+  <xacro:arg name="waist_initial_value"              default="0"/>
+  <xacro:arg name="shoulder_initial_value"           default="0"/>
+  <xacro:arg name="elbow_initial_value"              default="0"/>
+  <xacro:arg name="wrist_angle_initial_value"        default="0"/>
+  <xacro:arg name="wrist_rotate_initial_value"       default="0"/>
+  <xacro:arg name="finger_initial_value"             default="0"/>
   <xacro:property name="mesh_directory"             value="package://arm_sim_scenario/meshes/${robot_model}_meshes"/>
   <xacro:property name="urdf_loc"                   value="$(arg external_urdf_loc)"/>
@@ -24,20 +31,25 @@
   <xacro:property name="waist_limit_upper"          value="${pi - pi_offset}"/>
   <xacro:property name="waist_limit_vel"            value="${pi}"/>
+  <xacro:property name="waist_initial_value"         value="$(arg waist_initial_value)"/>
   <xacro:property name="shoulder_limit_effort"      value="18"/>
   <xacro:property name="shoulder_limit_lower"       value="${radians(-108)}"/>
   <xacro:property name="shoulder_limit_upper"       value="${radians(113)}"/>
   <xacro:property name="shoulder_limit_vel"         value="1"/>
+  <xacro:property name="shoulder_initial_value"      value="$(arg shoulder_initial_value)"/>
   <xacro:property name="elbow_limit_effort"         value="13"/>
   <xacro:property name="elbow_limit_lower"          value="${radians(-108)}"/>
   <xacro:property name="elbow_limit_upper"          value="${radians(93)}"/>
   <xacro:property name="elbow_limit_vel"            value="${pi}"/>
+  <xacro:property name="elbow_initial_value"         value="$(arg elbow_initial_value)"/>
   <xacro:property name="wrist_angle_limit_effort"   value="5"/>
   <xacro:property name="wrist_angle_limit_lower"    value="${radians(-100)}"/>
   <xacro:property name="wrist_angle_limit_upper"    value="${radians(123)}"/>
   <xacro:property name="wrist_angle_limit_vel"      value="${pi}"/>
+  <xacro:property name="wrist_angle_initial_value"   value="$(arg wrist_angle_initial_value)"/>
   <xacro:property name="wrist_rotate_limit_effort"  value="1"/>
   <xacro:property name="wrist_rotate_limit_lower"   value="${-pi + pi_offset}"/>
   <xacro:property name="wrist_rotate_limit_upper"   value="${pi - pi_offset}"/>
   <xacro:property name="wrist_rotate_limit_vel"     value="${pi}"/>
+  <xacro:property name="wrist_rotate_initial_value"  value="$(arg wrist_rotate_initial_value)"/>
   <xacro:property name="gripper_limit_vel"          value="${pi}"/>
   <xacro:property name="finger_limit_effort"        value="5"/>
@@ -45,4 +57,5 @@
   <xacro:property name="finger_limit_upper"         value="0.037"/>
   <xacro:property name="finger_limit_vel"           value="1"/>
+  <xacro:property name="finger_initial_value"        value="$(arg finger_initial_value)"/>
   <material name="interbotix_black">
     <texture filename="package://arm_sim_scenario/meshes/interbotix_black.png"/>
