Commit message: re-structure launch files

File: simulation/gazebo/arm_sim_scenario/config/srdf/wx200.srdf.xacro (robot description, xacro)
@@ -47,5 +47,5 @@
     <group_state name="Sleep" group="interbotix_arm">
         <joint name="elbow" value="1.55" />
-        <joint name="shoulder" value="-1.88" />
+        <joint name="shoulder" value="-1.60" />
         <joint name="waist" value="0" />
         <joint name="wrist_angle" value="0.8" />

File: simulation/gazebo/arm_sim_scenario/urdf/control.urdf.xacro (robot description, xacro)
@@ -135,5 +135,5 @@
         <robot_param>robot_description</robot_param>
         <robot_param_node>robot_state_publisher</robot_param_node>
-        <parameters>$(find arm_sim_scenario)/config/trajectory_controllers/${robot_model}_trajectory_controllers.yaml</parameters>
+        <parameters>$(find arm_sim_scenario)/config/trajectory_controllers/${robot_model}_trajectory_controllers_ignition.yaml</parameters>
       </plugin>
     </gazebo>
