Commit message: gazebo_static_camera: add static transform publisher

File: simulation/gazebo/gazebo_static_camera/models/camera.sdf.xacro (robot description, xacro)
@@ -4,8 +4,8 @@
   <xacro:arg name="image_height" default="240"/>
   <xacro:arg name="update_rate" default="5"/>
+  <xacro:arg name="camera_name" default="camera"/>
   <model name="camera">
     <static>true</static>
       <link name="link">
-        <pose>0.05 0.05 0.05 0 0 0</pose>
         <inertial>
           <mass>0.1</mass>
@@ -16,12 +16,6 @@
           </inertia>
         </inertial>
-        <collision name="collision">
-          <geometry>
-            <box>
-              <size>0.1 0.1 0.1</size>
-            </box>
-          </geometry>
-        </collision>
         <visual name="visual">
+          <pose>-0.05 -0.05 -0.05 0 0 0</pose>
           <geometry>
             <box>
@@ -32,4 +26,5 @@
         <sensor name="camera" type="camera">
           <camera>
+            <optical_frame_id>$(arg camera_name)_optical_frame</optical_frame_id>
             <horizontal_fov>1.047</horizontal_fov>
             <image>
