Commit message: cleanup

File: simulation/gazebo/arm_sim_scenario/config/control.urdf.xacro (robot description, xacro)
@@ -1,7 +1,5 @@
 <?xml version="1.0"?>
 <robot xmlns:xacro="http://ros.org/wiki/xacro">
-<xacro:macro name="panda_ros2_control" params="name initial_positions_file ros2_control_hardware_type">
-  <xacro:property name="initial_positions" value="${xacro.load_yaml(initial_positions_file)['initial_positions']}"/>
-    <ros2_control name="${name}" type="system">
+    <ros2_control name="HardwareInterface" type="system">
         <hardware>
             <xacro:if value="${ros2_control_hardware_type == 'mock_components'}">
@@ -18,7 +16,5 @@
               <param name="initial_value">${initial_positions['panda_joint1']}</param>
             </state_interface>
-            <state_interface name="velocity">
-              <param name="initial_value">0.0</param>
-            </state_interface>
+            <state_interface name="velocity" />
         </joint>
         <joint name="panda_joint2">
@@ -27,7 +23,5 @@
               <param name="initial_value">${initial_positions['panda_joint2']}</param>
             </state_interface>
-            <state_interface name="velocity">
-              <param name="initial_value">0.0</param>
-            </state_interface>
+            <state_interface name="velocity" />
         </joint>
         <joint name="panda_joint3">
@@ -36,7 +30,5 @@
               <param name="initial_value">${initial_positions['panda_joint3']}</param>
             </state_interface>
-            <state_interface name="velocity">
-              <param name="initial_value">0.0</param>
-            </state_interface>
+            <state_interface name="velocity" />
         </joint>
         <joint name="panda_joint4">
@@ -45,7 +37,5 @@
               <param name="initial_value">${initial_positions['panda_joint4']}</param>
             </state_interface>
-            <state_interface name="velocity">
-              <param name="initial_value">0.0</param>
-            </state_interface>
+            <state_interface name="velocity" />
         </joint>
         <joint name="panda_joint5">
@@ -54,7 +44,5 @@
               <param name="initial_value">${initial_positions['panda_joint5']}</param>
             </state_interface>
-            <state_interface name="velocity">
-              <param name="initial_value">0.0</param>
-            </state_interface>
+            <state_interface name="velocity" />
         </joint>
         <joint name="panda_joint6">
@@ -63,7 +51,5 @@
               <param name="initial_value">${initial_positions['panda_joint6']}</param>
             </state_interface>
-            <state_interface name="velocity">
-              <param name="initial_value">0.0</param>
-            </state_interface>
+            <state_interface name="velocity" />
         </joint>
         <joint name="panda_joint7">
@@ -72,7 +58,5 @@
               <param name="initial_value">${initial_positions['panda_joint7']}</param>
             </state_interface>
-            <state_interface name="velocity">
-              <param name="initial_value">0.0</param>
-            </state_interface>
+            <state_interface name="velocity" />
         </joint>
         <joint name="panda_finger_joint1">
@@ -104,4 +88,3 @@
       </gazebo>
     </xacro:if>
-</xacro:macro>
 </robot>

File: simulation/gazebo/arm_sim_scenario/config/panda.urdf.xacro (robot description, xacro)
@@ -2,27 +2,7 @@
 <robot name="panda" xmlns:xacro="http://www.ros.org/wiki/xacro">
     <xacro:arg name="ros2_control_hardware_type"                   default="${ros2_control_hardware_type}"/>
-    <xacro:arg name="prefix"                                       default="panda_"/>
-    <xacro:arg name="use_gripper"                                  default="true"/>
-    <xacro:arg name="joint1_initial_position"                      default="0.0"/>
-    <xacro:arg name="joint2_initial_position"                      default="-0.785"/>
-    <xacro:arg name="joint3_initial_position"                      default="0.0"/>
-    <xacro:arg name="joint4_initial_position"                      default="-2.356"/>
-    <xacro:arg name="joint5_initial_position"                      default="0.0"/>
-    <xacro:arg name="joint6_initial_position"                      default="1.571"/>
-    <xacro:arg name="joint7_initial_position"                      default="0.785"/>
-    <xacro:arg name="finger_joint1_initial_position"               default="0.0"/>
-    <xacro:arg name="finger_joint2_initial_position"               default="0.0"/>
+    <xacro:property name="initial_positions_file"                  value="$(find moveit_resources_panda_moveit_config)/config/initial_positions.yaml" />
+    <xacro:property name="initial_positions"                       value="${xacro.load_yaml(initial_positions_file)['initial_positions']}"/>
     <xacro:property name="ros2_control_hardware_type"              value="$(arg ros2_control_hardware_type)"/>
-    <xacro:property name="prefix"                                  value="$(arg prefix)"/>
-    <xacro:property name="use_gripper"                             value="$(arg use_gripper)"/>
-    <xacro:property name="joint1_initial_position"                 value="$(arg joint1_initial_position)"/>
-    <xacro:property name="joint2_initial_position"                 value="$(arg joint2_initial_position)"/>
-    <xacro:property name="joint3_initial_position"                 value="$(arg joint3_initial_position)"/>
-    <xacro:property name="joint4_initial_position"                 value="$(arg joint4_initial_position)"/>
-    <xacro:property name="joint5_initial_position"                 value="$(arg joint5_initial_position)"/>
-    <xacro:property name="joint6_initial_position"                 value="$(arg joint6_initial_position)"/>
-    <xacro:property name="joint7_initial_position"                 value="$(arg joint7_initial_position)"/>
-    <xacro:property name="finger_joint1_initial_position"          value="$(arg finger_joint1_initial_position)"/>
-    <xacro:property name="finger_joint2_initial_position"          value="$(arg finger_joint2_initial_position)"/>
     <link name="world"/>
     <joint name="panda_world" type="fixed">
@@ -31,19 +11,19 @@
         <child link="panda_link0" />
     </joint>
-    <link name="panda_link0">
-        <visual>
-            <geometry>
-                <mesh filename="package://moveit_resources_panda_description/meshes/visual/link0.dae" />
-            </geometry>
-        </visual>
-        <collision>
-            <geometry>
-                <mesh filename="package://moveit_resources_panda_description/meshes/collision/link0.stl" />
-            </geometry>
-        </collision>
-        <inertial>
-            <origin xyz="0 0 0" rpy="0 0 0" />
-            <mass value="3.06357" />
-            <inertia ixx="0.3" ixy="0.0" ixz="0.0" iyy="0.3" iyz="0.0" izz="0.3" />
+     <link name="panda_link0">
+        <visual>
+            <geometry>
+                <mesh filename="file://$(find moveit_resources_panda_description)/meshes/visual/link0.dae" />
+            </geometry>
+        </visual>
+        <collision>
+            <geometry>
+                <mesh filename="file://$(find moveit_resources_panda_description)/meshes/collision/link0.stl" />
+            </geometry>
+        </collision>
+        <inertial>
+          <origin xyz="-0.041018 -0.00014 0.049974" rpy="0 0 0" />
+          <mass value="0.629769"/>
+          <inertia ixx="0.00315" iyy="0.00388" izz="0.004285" ixy="8.2904E-7" ixz="0.00015" iyz="8.2299E-6"/>
         </inertial>
     </link>
@@ -51,16 +31,16 @@
         <visual>
             <geometry>
-                <mesh filename="package://moveit_resources_panda_description/meshes/visual/link1.dae" />
-            </geometry>
-        </visual>
-        <collision>
-            <geometry>
-                <mesh filename="package://moveit_resources_panda_description/meshes/collision/link1.stl" />
-            </geometry>
-        </collision>
-        <inertial>
-            <origin xyz="0 0 0" rpy="0 0 0" />
-            <mass value="2.34471" />
-            <inertia ixx="0.3" ixy="0.0" ixz="0.0" iyy="0.3" iyz="0.0" izz="0.3" />
+                <mesh filename="file://$(find moveit_resources_panda_description)/meshes/visual/link1.dae" />
+            </geometry>
+        </visual>
+        <collision>
+            <geometry>
+                <mesh filename="file://$(find moveit_resources_panda_description)/meshes/collision/link1.stl" />
+            </geometry>
+        </collision>
+        <inertial>
+          <origin xyz="0.003875 0.002081 -0.04762" rpy="0 0 0" />
+          <mass value="4.970684"/>
+          <inertia ixx="0.70337" iyy="0.70661" izz="0.009117" ixy="-0.000139" ixz="0.006772" iyz="0.019169"/>
         </inertial>
     </link>
@@ -72,20 +52,21 @@
         <axis xyz="0 0 1" />
         <limit effort="87" lower="-2.9671" upper="2.9671" velocity="2.3925" />
+        <dynamics D="1" K="7000" damping="0.003" friction="0.0" mu_coulomb="0" mu_viscous="16" />
     </joint>
     <link name="panda_link2">
         <visual>
             <geometry>
-                <mesh filename="package://moveit_resources_panda_description/meshes/visual/link2.dae" />
-            </geometry>
-        </visual>
-        <collision>
-            <geometry>
-                <mesh filename="package://moveit_resources_panda_description/meshes/collision/link2.stl" />
-            </geometry>
-        </collision>
-        <inertial>
-            <origin xyz="0 0 0" rpy="0 0 0" />
-            <mass value="2.36414" />
-            <inertia ixx="0.3" ixy="0.0" ixz="0.0" iyy="0.3" iyz="0.0" izz="0.3" />
+                <mesh filename="file://$(find moveit_resources_panda_description)/meshes/visual/link2.dae" />
+            </geometry>
+        </visual>
+        <collision>
+            <geometry>
+                <mesh filename="file://$(find moveit_resources_panda_description)/meshes/collision/link2.stl" />
+            </geometry>
+        </collision>
+        <inertial>
+          <origin xyz="-0.003141 -0.02872  0.003495" rpy="0 0 0" />
+          <mass value="0.646926"/>
+          <inertia ixx="0.007962" iyy="2.811E-2" izz="2.5995E-2" ixy="-3.925E-3" ixz="1.0254E-2" iyz="7.04E-4"/>
         </inertial>
     </link>
@@ -97,20 +78,21 @@
         <axis xyz="0 0 1" />
         <limit effort="87" lower="-1.8326" upper="1.8326" velocity="2.3925" />
+        <dynamics D="1" K="7000" damping="0.003" friction="0.0" mu_coulomb="0" mu_viscous="16" />
     </joint>
     <link name="panda_link3">
         <visual>
             <geometry>
-                <mesh filename="package://moveit_resources_panda_description/meshes/visual/link3.dae" />
-            </geometry>
-        </visual>
-        <collision>
-            <geometry>
-                <mesh filename="package://moveit_resources_panda_description/meshes/collision/link3.stl" />
-            </geometry>
-        </collision>
-        <inertial>
-            <origin xyz="0 0 0" rpy="0 0 0" />
-            <mass value="2.38050" />
-            <inertia ixx="0.3" ixy="0.0" ixz="0.0" iyy="0.3" iyz="0.0" izz="0.3" />
+                <mesh filename="file://$(find moveit_resources_panda_description)/meshes/visual/link3.dae" />
+            </geometry>
+        </visual>
+        <collision>
+            <geometry>
+                <mesh filename="file://$(find moveit_resources_panda_description)/meshes/collision/link3.stl" />
+            </geometry>
+        </collision>
+        <inertial>
+          <origin xyz="2.7518E-2 3.9252E-2 -6.6502E-2" rpy="0 0 0" />
+          <mass value="3.228604"/>
+          <inertia ixx="3.7242E-2" iyy="3.6155E-2" izz="1.083E-2" ixy="-4.761E-3" ixz="-1.1396E-2" iyz="-1.2805E-2"/>
         </inertial>
     </link>
@@ -122,20 +104,21 @@
         <axis xyz="0 0 1" />
         <limit effort="87" lower="-2.9671" upper="2.9671" velocity="2.3925" />
+        <dynamics D="1" K="7000" damping="0.003" friction="0.0" mu_coulomb="0" mu_viscous="16" />
     </joint>
     <link name="panda_link4">
         <visual>
             <geometry>
-                <mesh filename="package://moveit_resources_panda_description/meshes/visual/link4.dae" />
-            </geometry>
-        </visual>
-        <collision>
-            <geometry>
-                <mesh filename="package://moveit_resources_panda_description/meshes/collision/link4.stl" />
-            </geometry>
-        </collision>
-        <inertial>
-            <origin xyz="0 0 0" rpy="0 0 0" />
-            <mass value="2.42754" />
-            <inertia ixx="0.3" ixy="0.0" ixz="0.0" iyy="0.3" iyz="0.0" izz="0.3" />
+                <mesh filename="file://$(find moveit_resources_panda_description)/meshes/visual/link4.dae" />
+            </geometry>
+        </visual>
+        <collision>
+            <geometry>
+                <mesh filename="file://$(find moveit_resources_panda_description)/meshes/collision/link4.stl" />
+            </geometry>
+        </collision>
+        <inertial>
+          <origin xyz="-5.317E-2 1.04419E-1 2.7454E-2" rpy="0 0 0" />
+          <mass value="3.587895"/>
+          <inertia ixx="2.5853E-2" iyy="1.9552E-2" izz="2.8323E-2" ixy="7.796E-3" ixz="-1.332E-3" iyz="8.641E-3"/>
         </inertial>
     </link>
@@ -147,20 +130,21 @@
         <axis xyz="0 0 1" />
         <limit effort="87" lower="-3.1416" upper="0.0873" velocity="2.3925" />
+        <dynamics D="1" K="7000" damping="0.003" friction="0.0" mu_coulomb="0" mu_viscous="16" />
     </joint>
     <link name="panda_link5">
         <visual>
             <geometry>
-                <mesh filename="package://moveit_resources_panda_description/meshes/visual/link5.dae" />
-            </geometry>
-        </visual>
-        <collision>
-            <geometry>
-                <mesh filename="package://moveit_resources_panda_description/meshes/collision/link5.stl" />
-            </geometry>
-        </collision>
-        <inertial>
-            <origin xyz="0 0 0" rpy="0 0 0" />
-            <mass value="3.49611" />
-            <inertia ixx="0.3" ixy="0.0" ixz="0.0" iyy="0.3" iyz="0.0" izz="0.3" />
+                <mesh filename="file://$(find moveit_resources_panda_description)/meshes/visual/link5.dae" />
+            </geometry>
+        </visual>
+        <collision>
+            <geometry>
+                <mesh filename="file://$(find moveit_resources_panda_description)/meshes/collision/link5.stl" />
+            </geometry>
+        </collision>
+        <inertial>
+          <origin xyz="-1.1953E-2 4.1065E-2 -3.8437E-2" rpy="0 0 0" />
+          <mass value="1.225946"/>
+          <inertia ixx="3.5549E-2" iyy="2.9474E-2" izz="8.627E-3" ixy="-2.117E-3" ixz="-4.037E-3" iyz="2.29E-4"/>
         </inertial>
     </link>
@@ -172,20 +156,21 @@
         <axis xyz="0 0 1" />
         <limit effort="12" lower="-2.9671" upper="2.9671" velocity="2.8710" />
+        <dynamics D="1" K="7000" damping="0.003" friction="0.0" mu_coulomb="0" mu_viscous="16" />
     </joint>
     <link name="panda_link6">
         <visual>
             <geometry>
-                <mesh filename="package://moveit_resources_panda_description/meshes/visual/link6.dae" />
-            </geometry>
-        </visual>
-        <collision>
-            <geometry>
-                <mesh filename="package://moveit_resources_panda_description/meshes/collision/link6.stl" />
-            </geometry>
-        </collision>
-        <inertial>
-            <origin xyz="0 0 0" rpy="0 0 0" />
-            <mass value="1.46736" />
-            <inertia ixx="0.3" ixy="0.0" ixz="0.0" iyy="0.3" iyz="0.0" izz="0.3" />
+                <mesh filename="file://$(find moveit_resources_panda_description)/meshes/visual/link6.dae" />
+            </geometry>
+        </visual>
+        <collision>
+            <geometry>
+                <mesh filename="file://$(find moveit_resources_panda_description)/meshes/collision/link6.stl" />
+            </geometry>
+        </collision>
+        <inertial>
+          <origin xyz="6.0149E-2 -1.4117E-2 -1.0517E-2" rpy="0 0 0" />
+          <mass value="1.666555"/>
+          <inertia ixx="1.964E-3" iyy="4.354E-3" izz="5.433E-3" ixy="1.09E-4" ixz="-1.158E-3" iyz="3.41E-4"/>
         </inertial>
     </link>
@@ -197,20 +182,21 @@
         <axis xyz="0 0 1" />
         <limit effort="12" lower="-0.0873" upper="3.8223" velocity="2.8710" />
+        <dynamics D="1" K="7000" damping="0.003" friction="0.0" mu_coulomb="0" mu_viscous="16" />
     </joint>
     <link name="panda_link7">
         <visual>
             <geometry>
-                <mesh filename="package://moveit_resources_panda_description/meshes/visual/link7.dae" />
-            </geometry>
-        </visual>
-        <collision>
-            <geometry>
-                <mesh filename="package://moveit_resources_panda_description/meshes/collision/link7.stl" />
-            </geometry>
-        </collision>
-        <inertial>
-            <origin xyz="0 0 0" rpy="0 0 0" />
-            <mass value="0.45606" />
-            <inertia ixx="0.3" ixy="0.0" ixz="0.0" iyy="0.3" iyz="0.0" izz="0.3" />
+                <mesh filename="file://$(find moveit_resources_panda_description)/meshes/visual/link7.dae" />
+            </geometry>
+        </visual>
+        <collision>
+            <geometry>
+                <mesh filename="file://$(find moveit_resources_panda_description)/meshes/collision/link7.stl" />
+            </geometry>
+        </collision>
+        <inertial>
+          <origin xyz="1.0517E-2 -4.252E-3 6.1597E-2" rpy="0 0 0" />
+          <mass value="7.35522E-1"/>
+          <inertia ixx="1.2516E-2" iyy="1.0027E-2" izz="4.815E-3" ixy="-4.28E-4" ixz="-1.19E-3" iyz="-7.41E-4"/>
         </inertial>
     </link>
@@ -222,4 +208,5 @@
         <axis xyz="0 0 1" />
         <limit effort="12" lower="-2.9671" upper="2.9671" velocity="2.8710" />
+        <dynamics D="1" K="7000" damping="0.003" friction="0.0" mu_coulomb="0" mu_viscous="16" />
     </joint>
     <link name="panda_link8" />
@@ -238,16 +225,16 @@
         <visual>
             <geometry>
-                <mesh filename="package://moveit_resources_panda_description/meshes/visual/hand.dae" />
-            </geometry>
-        </visual>
-        <collision>
-            <geometry>
-                <mesh filename="package://moveit_resources_panda_description/meshes/collision/hand.stl" />
-            </geometry>
-        </collision>
-        <inertial>
-            <origin xyz="0 0 0" rpy="0 0 0" />
-            <mass value="0.67893" />
-            <inertia ixx="0.3" ixy="0.0" ixz="0.0" iyy="0.3" iyz="0.0" izz="0.3" />
+                <mesh filename="file://$(find moveit_resources_panda_description)/meshes/visual/hand.dae" />
+            </geometry>
+        </visual>
+        <collision>
+            <geometry>
+                <mesh filename="file://$(find moveit_resources_panda_description)/meshes/collision/hand.stl" />
+            </geometry>
+        </collision>
+        <inertial>
+          <origin xyz="-0.01 0 0.03" rpy="0 0 0" />
+          <mass value="0.73"/>
+          <inertia ixx="0.001" iyy="0.0025" izz="0.0017" ixy="0" ixz="0" iyz="0"/>
         </inertial>
     </link>
@@ -255,15 +242,16 @@
         <visual>
             <geometry>
-                <mesh filename="package://moveit_resources_panda_description/meshes/visual/finger.dae" />
-            </geometry>
-        </visual>
-        <collision>
-            <geometry>
-                <mesh filename="package://moveit_resources_panda_description/meshes/collision/finger.stl" />
-            </geometry>
-        </collision>
-        <inertial>
-            <mass value="0.01053" />
-            <inertia ixx="0.3" ixy="0.0" ixz="0.0" iyy="0.3" iyz="0.0" izz="0.3" />
+                <mesh filename="file://$(find moveit_resources_panda_description)/meshes/visual/finger.dae" />
+            </geometry>
+        </visual>
+        <collision>
+            <geometry>
+                <mesh filename="file://$(find moveit_resources_panda_description)/meshes/collision/finger.stl" />
+            </geometry>
+        </collision>
+        <inertial>
+          <origin xyz="0 0 0" rpy="0 0 0" />
+          <mass value="0.015"/>
+          <inertia ixx="2.375E-6" iyy="2.375E-6" izz="7.5E-7" ixy="0" ixz="0" iyz="0"/>
         </inertial>
     </link>
@@ -272,5 +260,5 @@
             <origin rpy="0 0 3.14159265359" xyz="0 0 0" />
             <geometry>
-                <mesh filename="package://moveit_resources_panda_description/meshes/visual/finger.dae" />
+                <mesh filename="file://$(find moveit_resources_panda_description)/meshes/visual/finger.dae" />
             </geometry>
         </visual>
@@ -278,10 +266,11 @@
             <origin rpy="0 0 3.14159265359" xyz="0 0 0" />
             <geometry>
-                <mesh filename="package://moveit_resources_panda_description/meshes/collision/finger.stl" />
-            </geometry>
-        </collision>
-        <inertial>
-            <mass value="0.01053" />
-            <inertia ixx="0.3" ixy="0.0" ixz="0.0" iyy="0.3" iyz="0.0" izz="0.3" />
+                <mesh filename="file://$(find moveit_resources_panda_description)/meshes/collision/finger.stl" />
+            </geometry>
+        </collision>
+        <inertial>
+          <origin xyz="0 0 0" rpy="0 0 0" />
+          <mass value="0.15"/>
+          <inertia ixx="2.375E-6" iyy="2.375E-6" izz="7.5E-7" ixy="0" ixz="0" iyz="0"/>
         </inertial>
     </link>
@@ -292,4 +281,5 @@
         <axis xyz="0 1 0" />
         <limit effort="20" lower="0.0" upper="0.04" velocity="0.2" />
+        <dynamics damping="0.3" />
     </joint>
     <joint name="panda_finger_joint2" type="prismatic">
@@ -300,10 +290,12 @@
         <limit effort="20" lower="0.0" upper="0.04" velocity="0.2" />
         <mimic joint="panda_finger_joint1" />
-    </joint>
-    <joint name="panda_finger_joint2_mimic" type="fixed">
+        <dynamics damping="0.3" />
+    </joint>
+     <joint name="panda_finger_joint2_mimic" type="fixed">
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